File: PICo-16f1765/PICo-16f1765.kicad_pcb (KiCad board)
At the start: 2 copper layers, 20.3 x 64.8 mm, 30 parts, among them IC1 PIC16F1765-I_P, IC2 CH340K, J1 Conn_01x06_Female, J2 Conn_01x09_Female, J3 Conn_01x09_Female, J4 USB_B_Micro, SW1 SW_Push, SW2 SW_Push, U1 LM1117-3.3, U2 LM1117S50TR_SOT223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

Commit message: fix: silks
Other:
- board text added: "3V3"
- board text added: "5V"
- board text added: "GND"
- board text added: "RA0"
- board text added: "RA1"
- board text added: "RA2"
- board text added: "RA3"
- board text added: "RA4"
- board text added: "RA5"
- board text added: "RC0"
- board text added: "RC1"
- board text added: "RC2"
- board text added: "RC3"
- board text added: "RC4"
- board text added: "RC5"
- board text added: "VCC"
- board text added: "Vin"
