File: PICo-16f1765/PICo-16f1765.sch (KiCad schematic (older format))
At the start: 24 parts, among them IC1 PIC16F1765-I_P, J1 Conn_01x06_Female, J2 Conn_01x09_Female, J3 Conn_01x09_Female, SW1 SW_Push, SW2 SW_Push, U1 LM1117-3.3, U2 LM1117S50TR_SOT223, X1 CSTLS8M00G53

Commit message: add: library files
Parts:
- C1, C2, C3, C4, C5: footprint (none) -> Capacitor_SMD:C_0201_0603Metric
- C6, C7: renamed from C?; footprint (none) -> Capacitor_SMD:C_0201_0603Metric
- D1: footprint (none) -> Diode_SMD:D_1206_3216Metric
- D2: footprint (none) -> LED_SMD:LED_0603_1608Metric
- IC1: footprint (none) -> Package_DIP:DIP-14_W7.62mm_Socket
- IC2: renamed from IC?; footprint (none) -> Package_SO:SSOP-10_3.9x4.9mm_P1.00mm
- J1: footprint (none) -> Connector_PinHeader_2.54mm:PinHeader_1x06_P2.54mm_Horizontal
- J2, J3: footprint (none) -> Connector_PinHeader_2.54mm:PinHeader_1x09_P2.54mm_Vertical
- R1, R2, R3: footprint (none) -> Resistor_SMD:R_0201_0603Metric
- gave numbers to parts that had none: 1
Changed lines of the file:
@@
 F 0 "IC1" H 3700 2565 50  0000 C CNN
 F 1 "PIC16F1765-I_P" H 3700 2474 50  0000 C CNN
-F 2 "" H 4500 2400 50  0001 L CNN
+F 2 "Package_DIP:DIP-14_W7.62mm_Socket" H 4500 2400 50  0001 L CNN
 F 3 "" H 4500 2300 50  0001 L CNN
 	1    3700 2000
@@
 F 0 "J1" H 1378 3426 50  0000 L CNN
 F 1 "Conn_01x06_Female" H 1378 3335 50  0000 L CNN
-F 2 "" H 1350 3450 50  0001 C CNN
+F 2 "Connector_PinHeader_2.54mm:PinHeader_1x06_P2.54mm_Horizontal" H 1350 3450 50  0001 C CNN
 F 3 "~" H 1350 3450 50  0001 C CNN
 	1    1350 3450
@@
 F 0 "R2" H 3520 3296 50  0000 L CNN
 F 1 "10k" H 3520 3205 50  0000 L CNN
-F 2 "" V 3380 3250 50  0001 C CNN
+F 2 "Resistor_SMD:R_0201_0603Metric" V 3380 3250 50  0001 C CNN
 F 3 "~" H 3450 3250 50  0001 C CNN
 	1    3450 3250
@@
 F 0 "R1" V 2943 7450 50  0000 C CNN
 F 1 "0" V 3034 7450 50  0000 C CNN
-F 2 "" V 3080 7450 50  0001 C CNN
+F 2 "Resistor_SMD:R_0201_0603Metric" V 3080 7450 50  0001 C CNN
 F 3 "~" H 3150 7450 50  0001 C CNN
 	1    3150 7450
@@
 F 0 "C2" H 2415 1296 50  0000 L CNN
 F 1 "0.1u" H 2415 1205 50  0000 L CNN
-F 2 "" H 2338 1100 50  0001 C CNN
+F 2 "Capacitor_SMD:C_0201_0603Metric" H 2338 1100 50  0001 C CNN
 F 3 "~" H 2300 1250 50  0001 C CNN
 	1    2300 1250
@@
 F 0 "C1" H 1715 6596 50  0000 L CNN
 F 1 "10u" H 1715 6505 50  0000 L CNN
-F 2 "" H 1638 6400 50  0001 C CNN
+F 2 "Capacitor_SMD:C_0201_0603Metric" H 1638 6400 50  0001 C CNN
 F 3 "~" H 1600 6550 50  0001 C CNN
 	1    1600 6550
@@
 F 0 "C3" H 2515 6596 50  0000 L CNN
 F 1 "10u" H 2515 6505 50  0000 L CNN
-F 2 "" H 2438 6400 50  0001 C CNN
+F 2 "Capacitor_SMD:C_0201_0603Metric" H 2438 6400 50  0001 C CNN
 F 3 "~" H 2400 6550 50  0001 C CNN
 	1    2400 6550
@@
 F 0 "C4" H 3265 6596 50  0000 L CNN
 F 1 "10u" H 3265 6505 50  0000 L CNN
-F 2 "" H 3188 6400 50  0001 C CNN
+F 2 "Capacitor_SMD:C_0201_0603Metric" H 3188 6400 50  0001 C CNN
 F 3 "~" H 3150 6550 50  0001 C CNN
 	1    3150 6550
@@
 F 0 "C5" H 4065 6596 50  0000 L CNN
 F 1 "10u" H 4065 6505 50  0000 L CNN
-F 2 "" H 3988 6400 50  0001 C CNN
+F 2 "Capacitor_SMD:C_0201_0603Metric" H 3988 6400 50  0001 C CNN
 F 3 "~" H 3950 6550 50  0001 C CNN
 	1    3950 6550
@@
 F 0 "D1" H 3600 6167 50  0000 C CNN
 F 1 "D_Schottky" H 3600 6076 50  0000 C CNN
-F 2 "" H 3600 5950 50  0001 C CNN
+F 2 "Diode_SMD:D_1206_3216Metric" H 3600 5950 50  0001 C CNN
 F 3 "~" H 3600 5950 50  0001 C CNN
 	1    3600 5950
@@
 F 0 "D2" V 4839 3132 50  0000 R CNN
 F 1 "LED" V 4748 3132 50  0000 R CNN
-F 2 "" H 4800 3250 50  0001 C CNN
+F 2 "LED_SMD:LED_0603_1608Metric" H 4800 3250 50  0001 C CNN
 F 3 "~" H 4800 3250 50  0001 C CNN
 	1    4800 3250
@@
 F 0 "R3" H 4870 3746 50  0000 L CNN
 F 1 "1k" H 4870 3655 50  0000 L CNN
-F 2 "" V 4730 3700 50  0001 C CNN
+F 2 "Resistor_SMD:R_0201_0603Metric" V 4730 3700 50  0001 C CNN
 F 3 "~" H 4800 3700 50  0001 C CNN
 	1    4800 3700
@@
 F 0 "J2" H 7378 2076 50  0000 L CNN
 F 1 "Conn_01x09_Female" H 7378 1985 50  0000 L CNN
-F 2 "" H 7350 2050 50  0001 C CNN
+F 2 "Connector_PinHeader_2.54mm:PinHeader_1x09_P2.54mm_Vertical" H 7350 2050 50  0001 C CNN
 F 3 "~" H 7350 2050 50  0001 C CNN
 	1    7350 2050
@@
 F 0 "J3" H 8292 1425 50  0000 C CNN
 F 1 "Conn_01x09_Female" H 8292 1516 50  0000 C CNN
-F 2 "" H 8400 2050 50  0001 C CNN
+F 2 "Connector_PinHeader_2.54mm:PinHeader_1x09_P2.54mm_Vertical" H 8400 2050 50  0001 C CNN
 F 3 "~" H 8400 2050 50  0001 C CNN
 	1    8400 2050
@@
 	8600 2450 9000 2450
 $Comp
-L Connector:USB_B_Micro J?
+L Connector:USB_B_Micro J4
 U 1 1 648497B0
 P 5900 5100
-F 0 "J?" H 5957 5567 50  0000 C CNN
+F 0 "J4" H 5957 5567 50  0000 C CNN
 F 1 "USB_B_Micro" H 5957 5476 50  0000 C CNN
 F 2 "" H 6050 5050 50  0001 C CNN
@@
 $EndComp
 $Comp
-L PICo-16f1765:CH340K IC?
+L PICo-16f1765:CH340K IC2
 U 1 1 6484A707
 P 7000 5300
-F 0 "IC?" H 7000 5765 50  0000 C CNN
+F 0 "IC2" H 7000 5765 50  0000 C CNN
 F 1 "CH340K" H 7000 5674 50  0000 C CNN
-F 2 "" H 7000 5550 50  0001 C CNN
+F 2 "Package_SO:SSOP-10_3.9x4.9mm_P1.00mm" H 7000 5550 50  0001 C CNN
 F 3 "" H 7000 5550 50  0001 C CNN
 	1    7000 5300
@@
 	6200 4750 6200 4900
 $Comp
-L power:GND #PWR?
+L power:GND #PWR027
 U 1 1 6486B023
 P 7500 6000
-F 0 "#PWR?" H 7500 5750 50  0001 C CNN
+F 0 "#PWR027" H 7500 5750 50  0001 C CNN
 F 1 "GND" H 7505 5827 50  0000 C CNN
 F 2 "" H 7500 6000 50  0001 C CNN
@@
 $EndComp
 $Comp
-L Device:C C?
+L Device:C C6
 U 1 1 64874DE7
 P 7500 5800
-F 0 "C?" H 7615 5846 50  0000 L CNN
+F 0 "C6" H 7615 5846 50  0000 L CNN
 F 1 "0.1u" H 7615 5755 50  0000 L CNN
-F 2 "" H 7538 5650 50  0001 C CNN
+F 2 "Capacitor_SMD:C_0201_0603Metric" H 7538 5650 50  0001 C CNN
 F 3 "~" H 7500 5800 50  0001 C CNN
 	1    7500 5800
@@
 $EndComp
 $Comp
-L Device:C C?
+L Device:C C7
 U 1 1 6487902E
 P 7950 5800
-F 0 "C?" H 8065 5846 50  0000 L CNN
+F 0 "C7" H 8065 5846 50  0000 L CNN
 F 1 "0.1u" H 8065 5755 50  0000 L CNN
-F 2 "" H 7988 5650 50  0001 C CNN
+F 2 "Capacitor_SMD:C_0201_0603Metric" H 7988 5650 50  0001 C CNN
 F 3 "~" H 7950 5800 50  0001 C CNN
 	1    7950 5800
@@
 $EndComp
 $Comp
-L power:GND #PWR?
+L power:GND #PWR028
 U 1 1 64879CBF
 P 7950 6000
-F 0 "#PWR?" H 7950 5750 50  0001 C CNN
+F 0 "#PWR028" H 7950 5750 50  0001 C CNN
 F 1 "GND" H 7955 5827 50  0000 C CNN
 F 2 "" H 7950 6000 50  0001 C CNN
@@
 NoConn ~ 7400 5500
 $Comp
-L power:GND #PWR?
+L power:GND #PWR026
 U 1 1 6485D830
 P 6400 6000
-F 0 "#PWR?" H 6400 5750 50  0001 C CNN
+F 0 "#PWR026" H 6400 5750 50  0001 C CNN
 F 1 "GND" H 6405 5827 50  0000 C CNN
 F 2 "" H 6400 6000 50  0001 C CNN
@@
 $EndComp
 $Comp
-L power:GND #PWR?
+L power:GND #PWR025
 U 1 1 64856AFE
 P 5900 6000
-F 0 "#PWR?" H 5900 5750 50  0001 C CNN
+F 0 "#PWR025" H 5900 5750 50  0001 C CNN
 F 1 "GND" H 5905 5827 50  0000 C CNN
 F 2 "" H 5900 6000 50  0001 C CNN

Commit message: feat: shape
Parts:
- removed X1: CSTLS8M00G53, symbol PICo-16f1765:CSTLS8M00G53
- added C8, C9: 22p, Capacitor_SMD:C_0603_1608Metric, symbol Device:C
- added J5, J6: Conn_01x02_Female, Connector_PinHeader_2.54mm:PinHeader_1x02_P2.54mm_Vertical, symbol Connector:Conn_01x02_Female
- added Y1: Crystal, Crystal:Crystal_HC49-U_Vertical, symbol Device:Crystal
- C1, C2, C3, C4, C5, C6, C7: footprint Capacitor_SMD:C_0201_0603Metric -> Capacitor_SMD:C_0603_1608Metric
- J4: footprint (none) -> PICo-16f1765:ZX62B5PA33
- JP1: footprint (none) -> Jumper:SolderJumper-3_P1.3mm_Bridged2Bar12_RoundedPad1.0x1.5mm
- R1, R2, R3: footprint Resistor_SMD:R_0201_0603Metric -> Resistor_SMD:R_0603_1608Metric
- SW1, SW2: footprint (none) -> PICo-16f1765:TVAF06A020BR
- U1, U2: footprint (none) -> Package_TO_SOT_SMD:SOT-223-3_TabPin2
Connections:
- net GND: now also C8.2, C9.2, J5.2 (Pin_2), J6.2 (Pin_2)
- net RA4: now also C9.1, Y1.2
- net RA5: now also C8.1, Y1.1
- net VCC: now also J5.1 (Pin_1), J6.1 (Pin_1)
Changed lines of the file:
@@
 $EndComp
-$Comp
-L PICo-16f1765:CSTLS8M00G53 X1
-U 1 1 64690561
-P 1350 1850
-F 0 "X1" H 1167 1385 50  0000 C CNN
-F 1 "CSTLS8M00G53" H 1167 1476 50  0000 C CNN
-F 2 "" H 1200 2250 50  0001 C CNN
-F 3 "" H 1200 2250 50  0001 C CNN
-	1    1350 1850
-	-1   0    0    1
-$EndComp
-Wire Wire Line
-	1950 2000 2100 2000
-Wire Wire Line
-	2100 2000 2100 1900
-Wire Wire Line
-	2100 1800 2100 1700
-Wire Wire Line
-	2100 1700 1950 1700
 $Comp
 L power:GND #PWR01
 U 1 1 64696731
-P 2000 2350
-F 0 "#PWR01" H 2000 2100 50  0001 C CNN
-F 1 "GND" H 2005 2177 50  0000 C CNN
-F 2 "" H 2000 2350 50  0001 C CNN
-F 3 "" H 2000 2350 50  0001 C CNN
-	1    2000 2350
-	1    0    0    -1
-$EndComp
-Wire Wire Line
-	1950 1850 2000 1850
+P 1350 2400
+F 0 "#PWR01" H 1350 2150 50  0001 C CNN
+F 1 "GND" H 1355 2227 50  0000 C CNN
+F 2 "" H 1350 2400 50  0001 C CNN
+F 3 "" H 1350 2400 50  0001 C CNN
+	1    1350 2400
+	1    0    0    -1
+$EndComp
 $Comp
 L power:GND #PWR019
@@
 	1    0    0    -1
 $EndComp
-Wire Wire Line
-	2000 1850 2000 2350
 $Comp
 L Connector:Conn_01x06_Female J1
@@
 	5450 2800 5450 1700
 Wire Wire Line
-	2100 1800 2750 1800
-Wire Wire Line
-	2100 1900 2750 1900
-Wire Wire Line
 	2300 2000 2750 2000
 Wire Wire Line
@@
 F 0 "SW1" H 3750 3335 50  0000 C CNN
 F 1 "SW_Push" H 3750 3244 50  0000 C CNN
-F 2 "" H 3750 3250 50  0001 C CNN
+F 2 "PICo-16f1765:TVAF06A020BR" H 3750 3250 50  0001 C CNN
 F 3 "~" H 3750 3250 50  0001 C CNN
 	1    3750 3050
@@
 F 0 "R2" H 3520 3296 50  0000 L CNN
 F 1 "10k" H 3520 3205 50  0000 L CNN
-F 2 "Resistor_SMD:R_0201_0603Metric" V 3380 3250 50  0001 C CNN
+F 2 "Resistor_SMD:R_0603_1608Metric" V 3380 3250 50  0001 C CNN
 F 3 "~" H 3450 3250 50  0001 C CNN
 	1    3450 3250
@@
 F 0 "SW2" H 3750 4385 50  0000 C CNN
 F 1 "SW_Push" H 3750 4294 50  0000 C CNN
-F 2 "" H 3750 4300 50  0001 C CNN
+F 2 "PICo-16f1765:TVAF06A020BR" H 3750 4300 50  0001 C CNN
 F 3 "~" H 3750 4300 50  0001 C CNN
 	1    3750 4100
@@
 F 0 "R1" V 2943 7450 50  0000 C CNN
 F 1 "0" V 3034 7450 50  0000 C CNN
-F 2 "Resistor_SMD:R_0201_0603Metric" V 3080 7450 50  0001 C CNN
+F 2 "Resistor_SMD:R_0603_1608Metric" V 3080 7450 50  0001 C CNN
 F 3 "~" H 3150 7450 50  0001 C CNN
 	1    3150 7450
@@
 F 0 "JP1" V 2796 5267 50  0000 L CNN
 F 1 "Jumper_3_Bridged12" V 2705 5267 50  0000 L CNN
-F 2 "" H 2750 5200 50  0001 C CNN
+F 2 "Jumper:SolderJumper-3_P1.3mm_Bridged2Bar12_RoundedPad1.0x1.5mm" H 2750 5200 50  0001 C CNN
 F 3 "~" H 2750 5200 50  0001 C CNN
 	1    2750 5200
@@
 F 0 "C2" H 2415 1296 50  0000 L CNN
 F 1 "0.1u" H 2415 1205 50  0000 L CNN
-F 2 "Capacitor_SMD:C_0201_0603Metric" H 2338 1100 50  0001 C CNN
+F 2 "Capacitor_SMD:C_0603_1608Metric" H 2338 1100 50  0001 C CNN
 F 3 "~" H 2300 1250 50  0001 C CNN
 	1    2300 1250
@@
 F 0 "U1" H 2050 6642 50  0000 C CNN
 F 1 "LM1117-3.3" H 2050 6551 50  0000 C CNN
-F 2 "" H 2050 6400 50  0001 C CNN
+F 2 "Package_TO_SOT_SMD:SOT-223-3_TabPin2" H 2050 6400 50  0001 C CNN
 F 3 "http://www.ti.com/lit/ds/symlink/lm1117.pdf" H 2050 6400 50  0001 C CNN
 	1    2050 6400
@@
 F 0 "U2" H 3600 6642 50  0000 C CNN
 F 1 "LM1117S50TR_SOT223" H 3600 6551 50  0000 C CNN
-F 2 "" H 3600 6400 50  0001 C CNN
+F 2 "Package_TO_SOT_SMD:SOT-223-3_TabPin2" H 3600 6400 50  0001 C CNN
 F 3 "http://www.ti.com/lit/ds/symlink/lm1117.pdf" H 3600 6400 50  0001 C CNN
 	1    3600 6400
@@
 F 0 "C1" H 1715 6596 50  0000 L CNN
 F 1 "10u" H 1715 6505 50  0000 L CNN
-F 2 "Capacitor_SMD:C_0201_0603Metric" H 1638 6400 50  0001 C CNN
+F 2 "Capacitor_SMD:C_0603_1608Metric" H 1638 6400 50  0001 C CNN
 F 3 "~" H 1600 6550 50  0001 C CNN
 	1    1600 6550
@@
 F 0 "C3" H 2515 6596 50  0000 L CNN
 F 1 "10u" H 2515 6505 50  0000 L CNN
-F 2 "Capacitor_SMD:C_0201_0603Metric" H 2438 6400 50  0001 C CNN
+F 2 "Capacitor_SMD:C_0603_1608Metric" H 2438 6400 50  0001 C CNN
 F 3 "~" H 2400 6550 50  0001 C CNN
 	1    2400 6550
@@
 F 0 "C4" H 3265 6596 50  0000 L CNN
 F 1 "10u" H 3265 6505 50  0000 L CNN
-F 2 "Capacitor_SMD:C_0201_0603Metric" H 3188 6400 50  0001 C CNN
+F 2 "Capacitor_SMD:C_0603_1608Metric" H 3188 6400 50  0001 C CNN
 F 3 "~" H 3150 6550 50  0001 C CNN
 	1    3150 6550
@@
 F 0 "C5" H 4065 6596 50  0000 L CNN
 F 1 "10u" H 4065 6505 50  0000 L CNN
-F 2 "Capacitor_SMD:C_0201_0603Metric" H 3988 6400 50  0001 C CNN
+F 2 "Capacitor_SMD:C_0603_1608Metric" H 3988 6400 50  0001 C CNN
 F 3 "~" H 3950 6550 50  0001 C CNN
 	1    3950 6550
@@
 F 0 "R3" H 4870 3746 50  0000 L CNN
 F 1 "1k" H 4870 3655 50  0000 L CNN
-F 2 "Resistor_SMD:R_0201_0603Metric" V 4730 3700 50  0001 C CNN
+F 2 "Resistor_SMD:R_0603_1608Metric" V 4730 3700 50  0001 C CNN
 F 3 "~" H 4800 3700 50  0001 C CNN
 	1    4800 3700
@@
 	1    0    0    -1
 $EndComp
-Text Label 8900 1650 0    50   ~ 0
-Vin
 Wire Wire Line
 	8900 1650 8600 1650
@@
 F 0 "J4" H 5957 5567 50  0000 C CNN
 F 1 "USB_B_Micro" H 5957 5476 50  0000 C CNN
-F 2 "" H 6050 5050 50  0001 C CNN
+F 2 "PICo-16f1765:ZX62B5PA33" H 6050 5050 50  0001 C CNN
 F 3 "~" H 6050 5050 50  0001 C CNN
 	1    5900 5100
@@
 F 0 "C6" H 7615 5846 50  0000 L CNN
 F 1 "0.1u" H 7615 5755 50  0000 L CNN
-F 2 "Capacitor_SMD:C_0201_0603Metric" H 7538 5650 50  0001 C CNN
+F 2 "Capacitor_SMD:C_0603_1608Metric" H 7538 5650 50  0001 C CNN
 F 3 "~" H 7500 5800 50  0001 C CNN
 	1    7500 5800
@@
 F 0 "C7" H 8065 5846 50  0000 L CNN
 F 1 "0.1u" H 8065 5755 50  0000 L CNN
-F 2 "Capacitor_SMD:C_0201_0603Metric" H 7988 5650 50  0001 C CNN
+F 2 "Capacitor_SMD:C_0603_1608Metric" H 7988 5650 50  0001 C CNN
 F 3 "~" H 7950 5800 50  0001 C CNN
 	1    7950 5800
@@
 Wire Wire Line
 	7400 5200 8350 5200
+$Comp
+L Device:Crystal Y1
+U 1 1 649327FA
+P 1350 1900
+F 0 "Y1" V 1304 2031 50  0000 L CNN
+F 1 "Crystal" V 1395 2031 50  0000 L CNN
+F 2 "Crystal:Crystal_HC49-U_Vertical" H 1350 1900 50  0001 C CNN
+F 3 "~" H 1350 1900 50  0001 C CNN
+	1    1350 1900
+	1    0    0    -1
+$EndComp
+$Comp
+L Device:C C8
+U 1 1 649379FC
+P 1100 2150
+F 0 "C8" H 1215 2196 50  0000 L CNN
+F 1 "22p" H 1215 2105 50  0000 L CNN
+F 2 "Capacitor_SMD:C_0603_1608Metric" H 1138 2000 50  0001 C CNN
+F 3 "~" H 1100 2150 50  0001 C CNN
+	1    1100 2150
+	1    0    0    -1
+$EndComp
+$Comp
+L Device:C C9
+U 1 1 64938EC5
+P 1600 2150
+F 0 "C9" H 1715 2196 50  0000 L CNN
+F 1 "22p" H 1715 2105 50  0000 L CNN
+F 2 "Capacitor_SMD:C_0603_1608Metric" H 1638 2000 50  0001 C CNN
+F 3 "~" H 1600 2150 50  0001 C CNN
+	1    1600 2150
+	1    0    0    -1
+$EndComp
+Wire Wire Line
+	1500 1900 1600 1900
+Wire Wire Line
+	1600 1900 1600 2000
+Wire Wire Line
+	1600 2300 1350 2300
+Wire Wire Line
+	1350 2300 1350 2400
+Wire Wire Line
+	1100 2300 1350 2300
+Connection ~ 1350 2300
+Wire Wire Line
+	1100 2000 1100 1900
+Wire Wire Line
+	1100 1900 1200 1900
+Wire Wire Line
+	1600 1900 2750 1900
+Connection ~ 1600 1900
+Wire Wire Line
+	1600 1800 1600 1450
+Wire Wire Line
+	1600 1450 1100 1450
+Wire Wire Line
+	1100 1450 1100 1900
+Wire Wire Line
+	1600 1800 2750 1800
+Connection ~ 1100 1900
+$Comp
+L Connector:Conn_01x02_Female J5
+U 1 1 6498876E
+P 9800 3600
+F 0 "J5" H 9828 3576 50  0000 L CNN
+F 1 "Conn_01x02_Female" H 9828 3485 50  0000 L CNN
+F 2 "Connector_PinHeader_2.54mm:PinHeader_1x02_P2.54mm_Vertical" H 9800 3600 50  0001 C CNN
+F 3 "~" H 9800 3600 50  0001 C CNN
+	1    9800 3600
+	1    0    0    -1
+$EndComp
+$Comp
+L power:VCC #PWR029
+U 1 1 6498A146
+P 9450 3600
+F 0 "#PWR029" H 9450 3450 50  0001 C CNN
+F 1 "VCC" H 9465 3773 50  0000 C CNN
+F 2 "" H 9450 3600 50  0001 C CNN
+F 3 "" H 9450 3600 50  0001 C CNN
+	1    9450 3600
+	1    0    0    -1
+$EndComp
+$Comp
+L power:GND #PWR030
+U 1 1 6498E6EF
+P 9450 3700
+F 0 "#PWR030" H 9450 3450 50  0001 C CNN
+F 1 "GND" H 9455 3527 50  0000 C CNN
+F 2 "" H 9450 3700 50  0001 C CNN
+F 3 "" H 9450 3700 50  0001 C CNN
+	1    9450 3700
+	1    0    0    -1
+$EndComp
+Wire Wire Line
+	9450 3600 9600 3600
+Wire Wire Line
+	9450 3700 9600 3700
+$Comp
+L Connector:Conn_01x02_Female J6
+U 1 1 649983E7
+P 9800 4300
+F 0 "J6" H 9828 4276 50  0000 L CNN
+F 1 "Conn_01x02_Female" H 9828 4185 50  0000 L CNN
+F 2 "Connector_PinHeader_2.54mm:PinHeader_1x02_P2.54mm_Vertical" H 9800 4300 50  0001 C CNN
+F 3 "~" H 9800 4300 50  0001 C CNN
+	1    9800 4300
+	1    0    0    -1
+$EndComp
+$Comp
+L power:VCC #PWR031
+U 1 1 649983ED
+P 9450 4300
+F 0 "#PWR031" H 9450 4150 50  0001 C CNN
+F 1 "VCC" H 9465 4473 50  0000 C CNN
+F 2 "" H 9450 4300 50  0001 C CNN
+F 3 "" H 9450 4300 50  0001 C CNN
+	1    9450 4300
+	1    0    0    -1
+$EndComp
+$Comp
+L power:GND #PWR032
+U 1 1 649983F3
+P 9450 4400
+F 0 "#PWR032" H 9450 4150 50  0001 C CNN
+F 1 "GND" H 9455 4227 50  0000 C CNN
+F 2 "" H 9450 4400 50  0001 C CNN
+F 3 "" H 9450 4400 50  0001 C CNN
+	1    9450 4400
+	1    0    0    -1
+$EndComp
+Wire Wire Line
+	9450 4300 9600 4300
+Wire Wire Line
+	9450 4400 9600 4400
+Text Label 8900 1650 0    50   ~ 0
+Vin
 $EndSCHEMATC

Commit message: fix: silks
Parts:
- removed J5, J6: Conn_01x02_Female, Connector_PinHeader_2.54mm:PinHeader_1x02_P2.54mm_Vertical, symbol Connector:Conn_01x02_Female
- added H1, H2, H3, H4: MountingHole, MountingHole:MountingHole_2.2mm_M2, symbol Mechanical:MountingHole
Changed lines of the file:
@@
 	1600 1800 2750 1800
 Connection ~ 1100 1900
+Text Label 8900 1650 0    50   ~ 0
+Vin
 $Comp
-L Connector:Conn_01x02_Female J5
-U 1 1 6498876E
-P 9800 3600
-F 0 "J5" H 9828 3576 50  0000 L CNN
-F 1 "Conn_01x02_Female" H 9828 3485 50  0000 L CNN
-F 2 "Connector_PinHeader_2.54mm:PinHeader_1x02_P2.54mm_Vertical" H 9800 3600 50  0001 C CNN
-F 3 "~" H 9800 3600 50  0001 C CNN
-	1    9800 3600
+L Mechanical:MountingHole H3
+U 1 1 648B4BDB
+P 10250 5150
+F 0 "H3" H 10350 5196 50  0000 L CNN
+F 1 "MountingHole" H 10350 5105 50  0000 L CNN
+F 2 "MountingHole:MountingHole_2.2mm_M2" H 10250 5150 50  0001 C CNN
+F 3 "~" H 10250 5150 50  0001 C CNN
+	1    10250 5150
 	1    0    0    -1
 $EndComp
 $Comp
-L power:VCC #PWR029
-U 1 1 6498A146
-P 9450 3600
-F 0 "#PWR029" H 9450 3450 50  0001 C CNN
-F 1 "VCC" H 9465 3773 50  0000 C CNN
-F 2 "" H 9450 3600 50  0001 C CNN
-F 3 "" H 9450 3600 50  0001 C CNN
-	1    9450 3600
+L Mechanical:MountingHole H1
+U 1 1 648BD151
+P 9450 5150
+F 0 "H1" H 9550 5196 50  0000 L CNN
+F 1 "MountingHole" H 9550 5105 50  0000 L CNN
+F 2 "MountingHole:MountingHole_2.2mm_M2" H 9450 5150 50  0001 C CNN
+F 3 "~" H 9450 5150 50  0001 C CNN
+	1    9450 5150
 	1    0    0    -1
 $EndComp
 $Comp
-L power:GND #PWR030
-U 1 1 6498E6EF
-P 9450 3700
-F 0 "#PWR030" H 9450 3450 50  0001 C CNN
-F 1 "GND" H 9455 3527 50  0000 C CNN
-F 2 "" H 9450 3700 50  0001 C CNN
-F 3 "" H 9450 3700 50  0001 C CNN
-	1    9450 3700
-	1    0    0    -1
-$EndComp
-Wire Wire Line
-	9450 3600 9600 3600
-Wire Wire Line
-	9450 3700 9600 3700
-$Comp
-L Connector:Conn_01x02_Female J6
-U 1 1 649983E7
-P 9800 4300
-F 0 "J6" H 9828 4276 50  0000 L CNN
-F 1 "Conn_01x02_Female" H 9828 4185 50  0000 L CNN
-F 2 "Connector_PinHeader_2.54mm:PinHeader_1x02_P2.54mm_Vertical" H 9800 4300 50  0001 C CNN
-F 3 "~" H 9800 4300 50  0001 C CNN
-	1    9800 4300
+L Mechanical:MountingHole H4
+U 1 1 648C1391
+P 10250 5450
+F 0 "H4" H 10350 5496 50  0000 L CNN
+F 1 "MountingHole" H 10350 5405 50  0000 L CNN
+F 2 "MountingHole:MountingHole_2.2mm_M2" H 10250 5450 50  0001 C CNN
+F 3 "~" H 10250 5450 50  0001 C CNN
+	1    10250 5450
 	1    0    0    -1
 $EndComp
 $Comp
-L power:VCC #PWR031
-U 1 1 649983ED
-P 9450 4300
-F 0 "#PWR031" H 9450 4150 50  0001 C CNN
-F 1 "VCC" H 9465 4473 50  0000 C CNN
-F 2 "" H 9450 4300 50  0001 C CNN
-F 3 "" H 9450 4300 50  0001 C CNN
-	1    9450 4300
+L Mechanical:MountingHole H2
+U 1 1 648C549C
+P 9450 5450
+F 0 "H2" H 9550 5496 50  0000 L CNN
+F 1 "MountingHole" H 9550 5405 50  0000 L CNN
+F 2 "MountingHole:MountingHole_2.2mm_M2" H 9450 5450 50  0001 C CNN
+F 3 "~" H 9450 5450 50  0001 C CNN
+	1    9450 5450
 	1    0    0    -1
 $EndComp
-$Comp
-L power:GND #PWR032
-U 1 1 649983F3
-P 9450 4400
-F 0 "#PWR032" H 9450 4150 50  0001 C CNN
-F 1 "GND" H 9455 4227 50  0000 C CNN
-F 2 "" H 9450 4400 50  0001 C CNN
-F 3 "" H 9450 4400 50  0001 C CNN
-	1    9450 4400
-	1    0    0    -1
-$EndComp
-Wire Wire Line
-	9450 4300 9600 4300
-Wire Wire Line
-	9450 4400 9600 4400
-Text Label 8900 1650 0    50   ~ 0
-Vin
 $EndSCHEMATC
